File: Wyse-converter.sch (KiCad schematic (older format))
At the start: 9 parts, among them J1 4P4C, U1 ProMicro, U2 ProMicro

Commit message: Fixed and working version
Parts:
- removed H1, H2: MountingHole, keyboard_parts:HOLE_M3, symbol Mechanical:MountingHole
- removed H5, H6: MountingHole_Pad, keyboard_parts:PIN_1, symbol Mechanical:MountingHole_Pad
Connections:
- net labels removed: RST
Other:
- moved on the sheet: H3, H4
Changed lines of the file:
@@
 DATA
-$Comp
-L Mechanical:MountingHole H2
-U 1 1 5F90B0FA
-P 3250 1400
-F 0 "H2" H 3350 1446 50  0000 L CNN
-F 1 "MountingHole" H 3350 1355 50  0000 L CNN
-F 2 "keyboard_parts:HOLE_M3" H 3250 1400 50  0001 C CNN
-F 3 "~" H 3250 1400 50  0001 C CNN
-	1    3250 1400
-	1    0    0    -1
-$EndComp
-$Comp
-L Mechanical:MountingHole H1
-U 1 1 5F90B8D4
-P 3250 1200
-F 0 "H1" H 3350 1246 50  0000 L CNN
-F 1 "MountingHole" H 3350 1155 50  0000 L CNN
-F 2 "keyboard_parts:HOLE_M3" H 3250 1200 50  0001 C CNN
-F 3 "~" H 3250 1200 50  0001 C CNN
-	1    3250 1200
-	1    0    0    -1
-$EndComp
 $Comp
 L Mechanical:MountingHole H3
 U 1 1 5F90C033
-P 3250 1600
-F 0 "H3" H 3350 1646 50  0000 L CNN
-F 1 "MountingHole" H 3350 1555 50  0000 L CNN
-F 2 "keyboard_parts:HOLE_M3" H 3250 1600 50  0001 C CNN
-F 3 "~" H 3250 1600 50  0001 C CNN
-	1    3250 1600
+P 3400 1300
+F 0 "H3" H 3500 1346 50  0000 L CNN
+F 1 "MountingHole" H 3500 1255 50  0000 L CNN
+F 2 "keyboard_parts:HOLE_M3" H 3400 1300 50  0001 C CNN
+F 3 "~" H 3400 1300 50  0001 C CNN
+	1    3400 1300
 	1    0    0    -1
 $EndComp
@@
 L Mechanical:MountingHole H4
 U 1 1 5F90C3D5
-P 3250 1800
-F 0 "H4" H 3350 1846 50  0000 L CNN
-F 1 "MountingHole" H 3350 1755 50  0000 L CNN
-F 2 "keyboard_parts:HOLE_M3" H 3250 1800 50  0001 C CNN
-F 3 "~" H 3250 1800 50  0001 C CNN
-	1    3250 1800
+P 3400 1500
+F 0 "H4" H 3500 1546 50  0000 L CNN
+F 1 "MountingHole" H 3500 1455 50  0000 L CNN
+F 2 "keyboard_parts:HOLE_M3" H 3400 1500 50  0001 C CNN
+F 3 "~" H 3400 1500 50  0001 C CNN
+	1    3400 1500
 	1    0    0    -1
 $EndComp
@@
 Text GLabel 3750 4550 0    50   Input ~ 0
 GND
-Text GLabel 3750 4450 0    50   Input ~ 0
-RST
-Text GLabel 5550 1950 0    50   Input ~ 0
-RST
-Text GLabel 5850 1750 2    50   Input ~ 0
-GND
-$Comp
-L Mechanical:MountingHole_Pad H5
-U 1 1 5F917DB4
-P 5650 1950
-F 0 "H5" V 5604 2100 50  0000 L CNN
-F 1 "MountingHole_Pad" V 5695 2100 50  0000 L CNN
-F 2 "keyboard_parts:PIN_1" H 5650 1950 50  0001 C CNN
-F 3 "~" H 5650 1950 50  0001 C CNN
-	1    5650 1950
-	0    1    1    0
-$EndComp
-$Comp
-L Mechanical:MountingHole_Pad H6
-U 1 1 5F9193F1
-P 5750 1750
-F 0 "H6" V 5987 1753 50  0000 C CNN
-F 1 "MountingHole_Pad" V 5896 1753 50  0000 C CNN
-F 2 "keyboard_parts:PIN_1" H 5750 1750 50  0001 C CNN
-F 3 "~" H 5750 1750 50  0001 C CNN
-	1    5750 1750
-	0    -1   -1   0
-$EndComp
 $EndSCHEMATC
